Commit message: Add matplotlibcpp and ability to plot the results of a simulation

File: data/urdfs/cart_pole.urdf (robot description, URDF)
Before this commit: robot physics, 3 links, 2 joints
Links:
- link pole: mass 0.2 -> 1
Joints:
- joint cart_to_pole: limit lower=-15 upper=15 effort=1000.0 velocity=5 -> (none)

Commit message: Clean up

File: data/urdfs/cart_pole.urdf (robot description, URDF)
Before this commit: robot physics, 3 links, 2 joints
Joints:
- joint slider_to_cart: limit lower=-15 upper=15 effort=1000.0 velocity=5 -> lower=-1000 upper=1000 effort=1000.0 velocity=5
