Commit message: Change simple.urdf joint limits

File: data/urdfs/simple.urdf (robot description, URDF)
Before this commit: robot compass_gait, 9 links, 8 joints
Joints:
- joint floating_base_x: limit lower=-1.57 upper=1.57 effort=100 velocity=100 -> lower=-100 upper=100 effort=100 velocity=100
- joint floating_base_z: limit lower=-1.57 upper=1.57 effort=100 velocity=100 -> lower=-100 upper=100 effort=100 velocity=100
- joint ground_rotation: limit lower=-1.57 upper=1.57 effort=100 velocity=100 -> lower=-100 upper=100 effort=100 velocity=100
- joint hip_joint: limit lower=-1.57 upper=1.57 effort=100 velocity=100 -> lower=-100 upper=100 effort=100 velocity=100
- joint left_foot_fixed: limit lower=-1.57 upper=1.57 effort=100 velocity=100 -> lower=-100 upper=100 effort=100 velocity=100
- joint left_hip_pitch: limit lower=-1.57 upper=1.57 effort=100 velocity=100 -> lower=-100 upper=100 effort=100 velocity=100
- joint right_foot_fixed: limit lower=-1.57 upper=1.57 effort=100 velocity=100 -> lower=-100 upper=100 effort=100 velocity=100
- joint right_hip_pitch: limit lower=-1.57 upper=1.57 effort=100 velocity=100 -> lower=-100 upper=100 effort=100 velocity=100
