Commit message: Remove 2nd link tree, move to using a mapping vector

File: data/urdfs/2_link_with_fixed.urdf (robot description, URDF)
Before this commit: robot 2_link, 3 links, 2 joints
Links:
- added link fixed_link, mass 1; visual sphere radius=.05
Joints:
- added joint fixed_joint: type fixed, parent link_1, child fixed_link, origin xyz=0 0 0 rpy=0 0 0, axis 0 0 1, limit lower=-100 upper=100 effort=100 velocity=100
- joint link_2: origin xyz=1 1 0 rpy=0 1.571 0 -> xyz=1 0 0 rpy=0 0 0; parent link_1 -> fixed_link

File: data/urdfs/3_link.urdf (robot description, URDF)
Before this commit: robot 2_link, 3 links, 2 joints
Links:
- added link link_3, mass 1; visual cylinder length=1 radius=.01
Joints:
- added joint link_3: type revolute, parent link_1, child link_3, origin xyz=1 0 0 rpy=0 1.571 0, axis 0 0 1, limit lower=-100 upper=100 effort=100 velocity=100
- joint link_2: origin xyz=1 1 0 rpy=0 1.571 0 -> xyz=0 0 0 rpy=0 0 0

File: data/urdfs/4_link.urdf (robot description, URDF)
Before this commit: robot 2_link, 3 links, 2 joints
Links:
- added link link_3, mass 1; visual cylinder length=1 radius=.01
- added link link_4, mass 1; visual cylinder length=1 radius=.01
Joints:
- added joint link_3: type revolute, parent link_1, child link_3, origin xyz=1 0 0 rpy=0 0 0, axis 0 0 1, limit lower=-100 upper=100 effort=100 velocity=100
- added joint link_4: type revolute, parent link_3, child link_4, origin xyz=1 0 0 rpy=0 0 0, axis 0 0 1, limit lower=-100 upper=100 effort=100 velocity=100
- joint link_2: origin xyz=1 1 0 rpy=0 1.571 0 -> xyz=1 0 0 rpy=0 0 0
