Commit message: Add functionality to deal with fixed joints
Should probably figure out a nicer way.

File: data/urdfs/2_link.urdf (robot description, URDF)
Before this commit: robot 2_link, 3 links, 2 joints
Links:
- added link fixed_link, mass 1; visual sphere radius=.05
Joints:
- added joint fixed_joint: type fixed, parent link_1, child fixed_link, origin xyz=0 0 0 rpy=0 0 0, axis 0 0 1, limit lower=-100 upper=100 effort=100 velocity=100
- joint link_2: parent link_1 -> fixed_link

Commit message: Update 2_link model

File: data/urdfs/2_link.urdf (robot description, URDF)
Before this commit: robot 2_link, 3 links, 2 joints
Joints:
- joint link_2: origin xyz=1 1 0 rpy=0 1.571 0 -> xyz=1 0 0 rpy=0 0 0

Commit message: Add autodiff and jacobian based methods

File: data/urdfs/2_link.urdf (robot description, URDF)
Before this commit: robot 2_link, 3 links, 2 joints
Links:
- added link end_effector, mass 0
Joints:
- added joint end_effector: type fixed, parent link_2, child end_effector, origin xyz=0 0 0 rpy=0 0 0, axis 0 0 0, limit lower=-100 upper=100 effort=100 velocity=100

File: data/urdfs/5_link.urdf (robot description, URDF)
Before this commit: robot 5_link, 6 links, 5 joints
Joints:
- joint link_3: parent link_1 -> link_2
- joint link_5: parent link_3 -> link_4
