Commit message: Add LEVENBERG_MARQUARDT method

File: data/urdfs/3_link.urdf (robot description, URDF)
Before this commit: robot 3_link, 4 links, 3 joints
Links:
- added link end_effector, mass 0
Joints:
- added joint end_effector: type fixed, parent link_3, child end_effector, origin xyz=0 0 0 rpy=0 0 0, axis 0 0 0, limit lower=-100 upper=100 effort=100 velocity=100

File: data/urdfs/4_link.urdf (robot description, URDF)
Before this commit: robot 4_link, 5 links, 4 joints
Links:
- added link end_effector, mass 0
Joints:
- added joint end_effector: type fixed, parent link_4, child end_effector, origin xyz=0 0 0 rpy=0 0 0, axis 0 0 0, limit lower=-100 upper=100 effort=100 velocity=100

File: data/urdfs/5_link.urdf (robot description, URDF)
Before this commit: robot 5_link, 6 links, 5 joints
Links:
- added link end_effector, mass 0
Joints:
- added joint end_effector: type fixed, parent link_5, child end_effector, origin xyz=0 0 0 rpy=0 0 0, axis 0 0 0, limit lower=-100 upper=100 effort=100 velocity=100
