Commit message: Begin implementation of geometric jacobians

File: data/urdfs/nugus.urdf (robot description, URDF)
Before this commit: robot nubots_nugus_hull, 21 links, 20 joints
Links:
- link head: mass 0.419 -> 4.2530
- link left_lower_arm: mass 0.26 -> 0
- link left_shoulder: mass 0.025434 -> 0
- link left_upper_arm: mass 0.297 -> 0
- link neck: mass 0.135 -> 0
- link right_lower_arm: mass 0.26 -> 0
- link right_shoulder: mass 0.025434 -> 0
- link right_upper_arm: mass 0.297 -> 0
- link torso: mass 2.539 -> 0
Joints:
- joint left_ankle_pitch: axis -1  0  0 -> 0 0 1; origin xyz=0    0.01 -0.2 rpy=3.14159  0      -3.14159 -> xyz=0.2 0 0 rpy=0 0 0
- joint left_ankle_roll: axis 0 -1  0 -> 0 0 1; origin xyz=0    0.04  0 rpy=-3.14159  0      -3.14159 -> xyz=0 0 0 rpy=1.571 0 0
- joint left_hip_pitch: axis 1  0  0 -> 0 0 1; origin xyz=0   -0.01  0 rpy=-0.05  0    0 -> xyz=0 0 0 rpy=-1.571 0 0
- joint left_hip_roll: axis 0 -1  0 -> 0 0 1; origin xyz=0    0   -0.06 rpy=0  0  0 -> xyz=0 0 -0.06 rpy=0  1.571  0
- joint left_hip_yaw: origin xyz=0     0.055  0 rpy=0       0       1.57079 -> xyz=0 0.055 0 rpy=0 0 0
- joint left_knee_pitch: axis 1  0  0 -> 0 0 1; origin xyz=0       0.00949 -0.18976 rpy=0.05  0    0 -> xyz=0.2 0 0 rpy=0 0 0
- joint right_ankle_pitch: axis -1  0  0 -> 0 0 1; origin xyz=0    0.01 -0.2 rpy=3.14159  0      -3.14159 -> xyz=0.2 0 0 rpy= 0 0 0
- joint right_ankle_roll: axis 0 -1  0 -> 0 0 1; origin xyz=0    0.04  0 rpy=-3.14159  0      -3.14159 -> xyz=0 0 0 rpy=1.571 0 0
- joint right_hip_pitch: axis 1  0  0 -> 0 0 1; origin xyz=0   -0.01  0.01 rpy=-0.05  0    0 -> xyz=0 0 0 rpy=-1.571 0 0
- joint right_hip_roll: axis 0 -1  0 -> 0 0 1; origin xyz=0    0   -0.06 rpy=0  0  0 -> xyz=0 0 -0.06 rpy=0  1.571  0
- joint right_hip_yaw: origin xyz=0    -0.055  0 rpy=0       0       1.57079 -> xyz=0    -0.055  0 rpy=0 0 0
- joint right_knee_pitch: axis 1  0  0 -> 0 0 1; origin xyz=0       0.00999 -0.19975 rpy=0.05  0    0 -> xyz=0.2 0 0 rpy=0 0 0

Commit message: Update IK and nugus model

File: data/urdfs/nugus.urdf (robot description, URDF)
Before this commit: robot nugus, 21 links, 20 joints
Links:
- added link left_camera, mass 1.01635e-15; collision box size=9.999999747378752e-06 1.0163475963054225e-05 9.999999747323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; visual mesh filename=left_camera_visual.stl
- added link left_foot_base, mass 1.01635e-23; collision box size=9.999999747378752e-06 1.0163475963054225e-05 9.999999747378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; visual mesh filename=left_foot_base_visual.stl
- added link right_camera, mass 1.01635e-23; collision box size=9.999999747378752e-06 1.0163475963054225e-05 9.999999747378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; visual mesh filename=right_camera_visual.stl
- added link right_foot_base, mass 1.01635e-23; collision box size=9.999999747378752e-06 1.0163475963054225e-05 9.999999747378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; visual mesh filename=right_foot_base_visual.stl
- link head: mass 4.2530 -> 0.473503; geometry collision box size=0.16223767679184675 0.15564338862895966 0.15779687464237213; visual mesh filename=head_visual.stl
- link left_ankle: mass 0.306 -> 0.329993; geometry collision box size=0.06627646926790476 0.09438799507915974 0.05529999919235706; visual mesh filename=left_ankle_visual.stl
- link left_foot: mass 0.205 -> 0.245581; geometry collision box size=0.05699313431978226 0.13158147037029266 0.21582108736038208; visual mesh filename=left_foot_visual.stl
- link left_hip_roll: mass 0.306 -> 0.395953; geometry collision box size=0.07245294097810984 0.05529999919235706 0.09385000355541706; visual mesh filename=left_hip_roll_visual.stl
- link left_hip_yaw: mass 0.067 -> 0.0594023; geometry collision box size=0.10850000381469727 0.09402551129460335 0.07350000609436158; visual mesh filename=left_hip_yaw_visual.stl
- link left_lower_arm: mass 0 -> 0.287325; geometry collision box size=0.08257202059030533 0.25829844921827316 0.050921617075800896; visual mesh filename=left_lower_arm_visual.stl
- link left_lower_leg: mass 0.177 -> 0.0893011; geometry collision box size=0.2292028944939375 0.03099999949336052 0.07800000160932541; visual mesh filename=left_lower_leg_visual.stl
- link left_shoulder: mass 0 -> 0.0845502; geometry collision box size=0.07999999821186066 0.08144209161400795 0.0793731525540351; visual mesh filename=left_shoulder_visual.stl
- link left_upper_arm: mass 0 -> 0.29923; geometry collision box size=0.22483809292316437 0.07902275025844574 0.08959516510367393; visual mesh filename=left_upper_arm_visual.stl
- link left_upper_leg: mass 0.387 -> 0.313357; geometry collision box size=0.2462693639099598 0.09347053803503513 0.0729999989271164; visual mesh filename=left_upper_leg_visual.stl
- link neck: mass 0 -> 0.165011; geometry collision box size=0.04019999876618385 0.05000000074505806 0.062835298711434; visual mesh filename=neck_visual.stl
- link right_ankle: mass 0.306 -> 0.329993; geometry collision box size=0.0656882356852293 0.094087990000844 0.05529999919235706; visual mesh filename=right_ankle_visual.stl
- link right_foot: mass 0.205 -> 0.245567; geometry collision box size=0.056986574083566666 0.13157938420772552 0.21582114696502686; visual mesh filename=right_foot_visual.stl
- link right_hip_roll: mass 0.306 -> 0.395953; geometry collision box size=0.06627646926790476 0.05529999919235706 0.09410000033676624; visual mesh filename=right_hip_roll_visual.stl
- link right_hip_yaw: mass 0.067 -> 0.0594022; geometry collision box size=0.10850000381469727 0.09402551129460335 0.07350000609436158; visual mesh filename=right_hip_yaw_visual.stl
- link right_lower_arm: mass 0 -> 0.28735; geometry collision box size=0.08257202059030533 0.2583179399371147 0.050956809893250465; visual mesh filename=right_lower_arm_visual.stl
- link right_lower_leg: mass 0.177 -> 0.0893011; geometry collision box size=0.22920288890600204 0.03099999949336052 0.07800000160932541; visual mesh filename=right_lower_leg_visual.stl
- link right_shoulder: mass 0 -> 0.0845501; geometry collision box size=0.07999999821186066 0.08146718889474869 0.07936178296804419; visual mesh filename=right_shoulder_visual.stl
- link right_upper_arm: mass 0 -> 0.299218; geometry collision box size=0.22482992708683014 0.07902275025844574 0.08959516510367393; visual mesh filename=right_upper_arm_visual.stl
- link right_upper_leg: mass 0.387 -> 0.313809; geometry collision box size=0.2462693639099598 0.09347053803503513 0.07300000265240669; visual mesh filename=right_upper_leg_visual.stl
- link torso: mass 0 -> 1.83264; geometry collision box size=0.13950913399457932 0.1899828165769577 0.2618043217808008; visual mesh filename=torso_visual.stl
Joints:
- added joint left_camera: type fixed, parent head, child left_camera, origin xyz=-0.0648803 -0.0699522 0.033795 rpy=1.5708 -1.63801e-13 -1.53589, axis 0 0 1, limit effort=1 velocity=20
- added joint left_foot_base: type fixed, parent left_foot, child left_foot_base, origin xyz=0.038 6.93889e-18 1.38778e-17 rpy=-4.52109e-30 -1.5708 0, axis 0 0 1, limit effort=1 velocity=20
- added joint right_camera: type fixed, parent head, child right_camera, origin xyz=-0.0648803 -0.0699522 -0.034205 rpy=1.5708 -1.63801e-13 -1.53589, axis 0 0 1, limit effort=1 velocity=20
- added joint right_foot_base: type fixed, parent right_foot, child right_foot_base, origin xyz=0.038 0 6.93889e-18 rpy=-1.26218e-29 -1.5708 0, axis 0 0 1, limit effort=1 velocity=20
- joint head_pitch: axis 1  0  0 -> 0 0 1; limit lower=-3.14159265359 upper=3.14159265359 effort=7.3 velocity=8.16814 -> lower=-3.14159 upper=3.14159 effort=1 velocity=20; origin xyz=0  0  0 rpy=0  0  0 -> xyz=-0.00024471 -0.000255294 0.0481 rpy=1.5708 1.5708 0
- joint left_ankle_pitch: limit lower=-3.14159265359 upper=3.14159265359 effort=10.0 velocity=5.75959 -> lower=-3.14159 upper=3.14159 effort=1 velocity=20; origin xyz=0.2 0 0 rpy=0 0 0 -> xyz=0.200203 -3.46945e-17 6.93889e-18 rpy=-3.05311e-15 5.55112e-17 -2.87748e-14
- joint left_ankle_roll: limit lower=-3.14159265359 upper=3.14159265359 effort=10.0 velocity=5.75959 -> lower=-3.14159 upper=3.14159 effort=1 velocity=20; origin xyz=0 0 0 rpy=1.571 0 0 -> xyz=0 0 6.93889e-18 rpy=1.5708 3.37316e-16 -3.88578e-16
- joint left_elbow_pitch: axis 1  0  0 -> 0 0 1; limit lower=-3.14159265359 upper=3.14159265359 effort=7.3 velocity=8.16814 -> lower=-3.14159 upper=3.14159 effort=1 velocity=20; origin xyz=-0.01    -0.19     0.03999 rpy=0  0  0 -> xyz=0.1575 -5.57465e-05 0.02695 rpy=-1.5708 1.5708 0
- joint left_hip_pitch: limit lower=-3.14159265359 upper=3.14159265359 effort=10.0 velocity=5.75959 -> lower=-3.14159 upper=3.14159 effort=1 velocity=20; origin xyz=0 0 0 rpy=-1.571 0 0 -> xyz=0 -6.93889e-18 -1.38778e-17 rpy=-1.5708 -1.29896e-14 3.34849e-14
- joint left_hip_roll: limit lower=-3.14159265359 upper=3.14159265359 effort=10.0 velocity=5.75959 -> lower=-3.14159 upper=3.14159 effort=1 velocity=20; origin xyz=0 0 -0.06 rpy=0  1.571  0 -> xyz=0.0221332 0 -0.0545 rpy=-4.55628e-30 1.5708 0
- joint left_hip_yaw: axis 0  0  1 -> 0 0 1; limit lower=-3.14159265359 upper=3.14159265359 effort=10.0 velocity=5.75959 -> lower=-3.14159 upper=3.14159 effort=1 velocity=20; origin xyz=0 0.055 0 rpy=0 0 0 -> xyz=7.63278e-17 0.055 0 rpy=-5.43064e-25 -3.21985e-24 6.16346e-16
- joint left_knee_pitch: limit lower=-3.14159265359 upper=3.14159265359 effort=10.0 velocity=5.75959 -> lower=-3.14159 upper=3.14159 effort=1 velocity=20; origin xyz=0.2 0 0 rpy=0 0 0 -> xyz=0.206046 0.0569501 -1.44745e-14 rpy=-4.42146e-14 -3.94129e-15 -1.40554e-13
- joint left_shoulder_pitch: axis 1  0  0 -> 0 0 1; limit lower=-3.14159265359 upper=3.14159265359 effort=7.3 velocity=8.16814 -> lower=-3.14159 upper=3.14159 effort=1 velocity=20; origin xyz=0.005  0.115  0.18 rpy=-1.57079  0       1.57079 -> xyz=-5.659e-18 0.077 0.17725 rpy=-1.5708 1.5708 0
- joint left_shoulder_roll: axis 0  0  1 -> 0 0 1; limit lower=-3.14159265359 upper=3.14159265359 effort=7.3 velocity=8.16814 -> lower=-3.14159 upper=3.14159 effort=1 velocity=20; origin xyz=0.015  0     0.005 rpy=1.57079  0       0 -> xyz=0 -0.0100012 0.0479124 rpy=1.5708 3.06087e-14 -1.5708
- joint neck_yaw: axis 0  0  1 -> 0 0 1; limit lower=-3.14159265359 upper=3.14159265359 effort=7.3 velocity=8.16814 -> lower=-3.14159 upper=3.14159 effort=1 velocity=20; origin xyz=0    0    0.26 rpy=0       0       1.57079 -> xyz=-0.008 2.09034e-16 0.20825 rpy=-1.1045e-15 2.10942e-15 -3.14159
- joint right_ankle_pitch: limit lower=-3.14159265359 upper=3.14159265359 effort=10.0 velocity=5.75959 -> effort=1 velocity=20; origin xyz=0.2 0 0 rpy= 0 0 0 -> xyz=0.200203 4.85723e-17 -6.93889e-18 rpy=1.88738e-15 -2.83277e-16 1.06524e-14
- joint right_ankle_roll: limit lower=-3.14159265359 upper=3.14159265359 effort=10.0 velocity=5.75959 -> lower=-3.14159 upper=3.14159 effort=1 velocity=20; origin xyz=0 0 0 rpy=1.571 0 0 -> xyz=1.27676e-15 1.249e-16 -8.46545e-16 rpy=1.5708 -1.11022e-15 7.94382e-15
- joint right_elbow_pitch: axis 1  0  0 -> 0 0 1; limit lower=-3.14159265359 upper=3.14159265359 effort=7.3 velocity=8.16814 -> lower=-3.14159 upper=3.14159 effort=1 velocity=20; origin xyz=0.01 -0.19  0.04 rpy=0  0  0 -> xyz=0.1575 5.57465e-05 0.02695 rpy=-1.5708 1.5708 0
- joint right_hip_pitch: limit lower=-3.14159265359 upper=3.14159265359 effort=10.0 velocity=5.75959 -> lower=-3.14159 upper=3.14159 effort=1 velocity=20; origin xyz=0 0 0 rpy=-1.571 0 0 -> xyz=-1.249e-16 0 3.81639e-17 rpy=-1.5708 -1.66533e-16 3.79139e-29
- joint right_hip_roll: limit lower=-3.14159265359 upper=3.14159265359 effort=10.0 velocity=5.75959 -> lower=-3.14159 upper=3.14159 effort=1 velocity=20; origin xyz=0 0 -0.06 rpy=0  1.571  0 -> xyz=0.0221332 0 -0.0545 rpy=1.36238e-31 1.5708 0
- joint right_hip_yaw: axis 0  0  1 -> 0 0 1; limit lower=-3.14159265359 upper=3.14159265359 effort=10.0 velocity=5.75959 -> lower=-3.14159 upper=3.14159 effort=1 velocity=20; origin xyz=0    -0.055  0 rpy=0 0 0 -> xyz=-6.93889e-18 -0.055 -5.55112e-17 rpy=-1.44515e-26 2.05167e-26 2.3927e-15
- joint right_knee_pitch: limit lower=-3.14159265359 upper=3.14159265359 effort=10.0 velocity=5.75959 -> lower=-3.14159 upper=3.14159 effort=1 velocity=20; origin xyz=0.2 0 0 rpy=0 0 0 -> xyz=0.206046 0.0569501 -7.16788e-15 rpy=-7.0209e-15 3.9968e-14 -5.66214e-15
- joint right_shoulder_pitch: axis 1  0  0 -> 0 0 1; limit lower=-3.14159265359 upper=3.14159265359 effort=7.3 velocity=8.16814 -> lower=-3.14159 upper=3.14159 effort=1 velocity=20; origin xyz=0.005 -0.115  0.18 rpy=-1.57079  0       1.57079 -> xyz=-3.55526e-17 -0.077 0.17725 rpy=-1.5708 1.5708 0
- joint right_shoulder_roll: axis 0  0  1 -> 0 0 1; limit lower=-3.14159265359 upper=3.14159265359 effort=7.3 velocity=8.16814 -> lower=-3.14159 upper=3.14159 effort=1 velocity=20; origin xyz=-0.015  0     0.005 rpy=1.57079  0       0 -> xyz=0 -0.0100012 -0.0479124 rpy=1.5708 -4.32987e-15 -1.5708
